File: BLE_LED_Dongle/BLE_LED_Dongle.kicad_sch (KiCad schematic)
At the start: 17 parts, among them J1 Conn_01x04, J2 Conn_02x08_Counter_Clockwise, U1 nRF52810-QCxx, Y1 Crystal, Y2 Crystal_GND23

Commit message: progress: PCB Part Placement of Patterns Complete
Parts:
- C5: footprint (none) -> Capacitor_SMD:C_0402_1005Metric
- U1: footprint Crystal:Crystal_SMD_0603-4Pin_6.0x3.5mm_HandSoldering -> Package_DFN_QFN:QFN-32-1EP_5x5mm_P0.5mm_EP3.6x3.6mm
Changed lines of the file:
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@@
+	)
+	(symbol
+		(lib_id "MCU_Nordic:nRF52810-QCxx")
+		(at 111.76 92.71 0)
+		(unit 1)
+		(exclude_from_sim no)
+		(in_bom yes)
+		(on_board yes)
+		(dnp no)
+		(fields_autoplaced yes)
+		(property "Reference" "U1"
+			(at 113.9033 118.11 0)
+			(effects
+				(font
+					(size 1.27 1.27)
+				)
+				(justify left)
+			)
+		)
+		(property "Value" "nRF52810-QCxx"
+			(at 113.9033 120.65 0)
+			(effects
+				(font
+					(size 1.27 1.27)
+				)
+				(justify left)
+			)
+		)
+		(property "Footprint" "Package_DFN_QFN:QFN-32-1EP_5x5mm_P0.5mm_EP3.6x3.6mm"
+			(at 111.76 127 0)
+			(effects
+				(font
+					(size 1.27 1.27)
+				)
+				(hide yes)
+			)
+		)
+		(property "Datasheet" "http://infocenter.nordicsemi.com/pdf/nRF52810_PS_v1.1.pdf"
+			(at 99.06 87.63 0)
+			(effects
+				(font
+					(size 1.27 1.27)
+				)
+				(hide yes)
+			)
+		)
+		(property "Description" "Multiprotocol BLE/2.4GHz Cortex-M4 SoC, QFN-32"
+			(at 111.76 92.71 0)
+			(effects
+				(font
+					(size 1.27 1.27)
+				)
+				(hide yes)
+			)
+		)
+		(pin "24"
+		)
+		(pin "19"
+		)
+		(pin "23"
+		)
+		(pin "22"
+		)
+		(pin "20"
+		)
+		(pin "16"
+		)
+		(pin "17"
+		)
+		(pin "1"
+		)
+		(pin "30"
+		)
+		(pin "25"
+		)
+		(pin "9"
+		)
+		(pin "29"
+		)
+		(pin "18"
+		)
+		(pin "21"
+		)
+		(pin "33"
+		)
+		(pin "31"
+		)
+		(pin "2"
+		)
+		(pin "32"
+		)
+		(pin "27"
+		)
+		(pin "3"
+		)
+		(pin "4"
+		)
+		(pin "28"
+		)
+		(pin "8"
+		)
+		(pin "11"
+		)
+		(pin "12"
+		)
+		(pin "13"
+		)
+		(pin "10"
+		)
+		(pin "26"
+		)
+		(pin "6"
+		)
+		(pin "5"
+		)
+		(pin "14"
+		)
+		(pin "15"
+		)
+		(pin "7"
+		)
+		(instances
+			(project ""
+				(path "/c8989c58-82e7-4a6e-815d-1abbb9dc8f72"
+					(reference "U1")
+					(unit 1)
+				)
+			)
+		)
 	)
 	(symbol
@@
 			)
 		)
-		(property "Footprint" ""
+		(property "Footprint" "Capacitor_SMD:C_0402_1005Metric"
 			(at 89.8652 66.04 0)
 			(effects
@@
 					(unit 1)
 				)
-			)
-		)
-	)
-	(symbol
-		(lib_id "MCU_Nordic:nRF52810-QCxx")
-		(at 111.76 92.71 0)
-		(unit 1)
-		(exclude_from_sim no)
-		(in_bom yes)
-		(on_board yes)
-		(dnp no)
-		(fields_autoplaced yes)
-		(property "Reference" "U1"
-			(at 113.9033 118.11 0)
-			(effects
-				(font
-					(size 1.27 1.27)
-				)
-				(justify left)
-			)
-		)
-		(property "Value" "nRF52810-QCxx"
-			(at 113.9033 120.65 0)
-			(effects
-				(font
-					(size 1.27 1.27)
-				)
-				(justify left)
-			)
-		)
-		(property "Footprint" "Crystal:Crystal_SMD_0603-4Pin_6.0x3.5mm_HandSoldering"
-			(at 111.76 127 0)
-			(effects
-				(font
-					(size 1.27 1.27)
-				)
-				(hide yes)
-			)
-		)
-		(property "Datasheet" "http://infocenter.nordicsemi.com/pdf/nRF52810_PS_v1.1.pdf"
-			(at 99.06 87.63 0)
-			(effects
-				(font
-					(size 1.27 1.27)
-				)
-				(hide yes)
-			)
-		)
-		(property "Description" "Multiprotocol BLE/2.4GHz Cortex-M4 SoC, QFN-32"
-			(at 111.76 92.71 0)
-			(effects
-				(font
-					(size 1.27 1.27)
-				)
-				(hide yes)
-			)
-		)
-		(pin "22"
-		)
-		(pin "2"
-		)
-		(pin "16"
-		)
-		(pin "10"
-		)
-		(pin "20"
-		)
-		(pin "8"
-		)
-		(pin "1"
-		)
-		(pin "5"
-		)
-		(pin "17"
-		)
-		(pin "24"
-		)
-		(pin "30"
-		)
-		(pin "32"
-		)
-		(pin "26"
-		)
-		(pin "18"
-		)
-		(pin "14"
-		)
-		(pin "23"
-		)
-		(pin "31"
-		)
-		(pin "33"
-		)
-		(pin "3"
-		)
-		(pin "19"
-		)
-		(pin "29"
-		)
-		(pin "9"
-		)
-		(pin "4"
-		)
-		(pin "21"
-		)
-		(pin "25"
-		)
-		(pin "6"
-		)
-		(pin "7"
-		)
-		(pin "11"
-		)
-		(pin "12"
-		)
-		(pin "13"
-		)
-		(pin "15"
-		)
-		(pin "27"
-		)
-		(pin "28"
-		)
-		(instances
-			(project ""
-				(path "/c8989c58-82e7-4a6e-815d-1abbb9dc8f72"
-					(reference "U1")
-					(unit 1)
-				)

Commit message: progress: board 1 complete, board 2 schematics in progress.
Parts:
- C1, C2, C3, C4: LCSC (none) -> C76948
- C10: LCSC (none) -> C23733
- C11: LCSC (none) -> C327032
- C5, C8, C9: LCSC (none) -> C1525
- C6: LCSC (none) -> C26409
- C7: LCSC (none) -> C14445
- J1: LCSC (none) -> C492412
- L1: LCSC (none) -> C98062
- U1: LCSC (none) -> C519278
- Y1: LCSC (none) -> C97606
- Y2: LCSC (none) -> C2965582
Connections:
- net LED_Matrix1/DIN: now also J2.3 (Pin_2); no longer J2.2 (Pin_2)
- net Power/EN_5V: now also J2.4 (Pin_15); no longer J2.15 (Pin_15)
- net at J2.10 (Pin_12): now also U1.14 (P0.18)
- net at J2.11 (Pin_6): now also U1.15 (P0.20); no longer U1.16 (P0.21/~{RESET})
- net at J2.12 (Pin_11): now also U1.16 (P0.21/~{RESET}); no longer U1.14 (P0.18)
- net at U1.12 (P0.15): now also J2.8 (Pin_13); no longer J2.13 (Pin_13)
- net at U1.10 (P0.12): now also J2.6 (Pin_14); no longer J2.14 (Pin_14)
- net at J2.16: now also U1.27 (P0.28/AIN4); no longer U1.5 (P0.05/AIN3)
- net at U1.8 (P0.10): now also J2.5 (Pin_3); no longer J2.3 (Pin_3)
- net at U1.11 (P0.14): now also J2.7 (Pin_4); no longer J2.4 (Pin_4)
- net at U1.13 (P0.16): now also J2.9 (Pin_5); no longer J2.5 (Pin_5)
- net at U1.26 (P0.25): now also J2.13 (Pin_7); no longer J2.7 (Pin_7)
- net at U1.28 (P0.30/AIN6): now also J2.15 (Pin_8); no longer J2.8 (Pin_8)
- new net: J2.2 (Pin_16), U1.5 (P0.05/AIN3)
