File: SPLD_Test/_autosave-SPLD_Test.kicad_sch (KiCad schematic)
At the start: 26 parts, among them J1 USB_C_Receptacle_PowerOnly_6P, J2 Conn_02x09_Top_Bottom, J3 Conn_02x09_Top_Bottom, J4 SPI OLED 1.3in, J5 SWD, J6 Conn_02x09_Top_Bottom, SW1 SW_MEC_5E, SW2 SW_MEC_5E, SW3 SW_MEC_5E, SW4 SW_MEC_5E, U1 ATF1502ASV-xAx44, U10 EA8105, U2 CA56-12CGKWA, U3 STM32F030K6Tx

Commit message: progress: CPLD Circuit schmatics complete & pattern placement in progress
Parts:
- C1: renamed from C9; now in the parts list
- C2: renamed from C1; now in the parts list
- J1: renamed from J4; footprint (none) -> Connector_PinSocket_2.54mm:PinSocket_1x07_P2.54mm_Vertical
- J3: renamed from J6; footprint (none) -> Connector_PinSocket_2.54mm:PinSocket_2x09_P2.54mm_Vertical
- J4: renamed from J5; footprint (none) -> Connector_PinSocket_2.54mm:PinSocket_1x06_P2.54mm_Vertical
- L1: renamed from L4; now in the parts list
- R1: renamed from R4; now in the parts list
- R2: renamed from R63; now in the parts list
- R3: renamed from R5; now in the parts list
- R4: renamed from R65; now in the parts list
- R5: renamed from R61; now in the parts list
- R6: renamed from R1; now in the parts list
- R7: renamed from R69; now in the parts list
- R8: renamed from R2; now in the parts list
- R9: renamed from R3; now in the parts list
- U2: renamed from U10; now in the parts list
- renumbered J1 to J2, J3 to J5, J2 to J6, SW4 to SW1, SW1 to SW3, SW3 to SW4, U3 to U1, U2 to U3, U1 to U4
