File: SPLD_Test/SPLD_Test.kicad_pcb (KiCad board)
At the start: 2 copper layers, 100 x 77 mm, 26 parts, among them J1 SPI OLED 1.3in, J2 USB_C_Receptacle_PowerOnly_6P, J3 Conn_02x09_Top_Bottom, J4 SWD, J5 Conn_02x09_Top_Bottom, J6 Conn_02x09_Top_Bottom, SW1 SW_MEC_5E, SW2 SW_MEC_5E, SW3 SW_MEC_5E, SW4 SW_MEC_5E, U1 STM32F030K6Tx, U2 EA8105, U3 CA56-12CGKWA, U4 ATF1502ASV-xAx44

Commit message: progress: CPLD Board complete
Parts:
- added R10: 10k, Resistor_SMD:R_0402_1005Metric_Pad0.72x0.64mm_HandSolder, B.Cu at (178.2, 51.0)
- added R11: 10k, Resistor_SMD:R_0402_1005Metric_Pad0.72x0.64mm_HandSolder, B.Cu at (178.2, 54.6)
- added R12: 10k, Resistor_SMD:R_0402_1005Metric_Pad0.72x0.64mm_HandSolder, B.Cu at (178.2, 57.4)
- added R13: 10k, Resistor_SMD:R_0402_1005Metric_Pad0.72x0.64mm_HandSolder, B.Cu at (178.2, 60.2)
- added R14: 10k, Resistor_SMD:R_0402_1005Metric_Pad0.72x0.64mm_HandSolder, B.Cu at (178.2, 61.6)
- added R15: 10k, Resistor_SMD:R_0402_1005Metric_Pad0.72x0.64mm_HandSolder, B.Cu at (178.2, 52.4)
- added R16: 10k, Resistor_SMD:R_0402_1005Metric_Pad0.72x0.64mm_HandSolder, B.Cu at (178.2, 56.0)
- added R17: 10k, Resistor_SMD:R_0402_1005Metric_Pad0.72x0.64mm_HandSolder, B.Cu at (178.2, 58.8)
Connections:
- U3 pad 1: /I/O11 -> Net-(U3-e)
- U3 pad 10: /I/O12 -> Net-(U3-f)
- U3 pad 11: /I/O6 -> Net-(U3-a)
- U3 pad 2: /I/O10 -> Net-(U3-d)
- U3 pad 3: /I/O14 -> Net-(U3-DPX)
- U3 pad 4: /I/O8 -> Net-(U3-c)
- U3 pad 5: /I/O13 -> Net-(U3-g)
- U3 pad 7: /I/O7 -> Net-(U3-b)
Routing:
- net +3.3V: track 0.00 -> 407.2 mm, vias 0 -> 5
- net /I/O18: track 0.00 -> 140.0 mm, vias 0 -> 1
- net /I/O15: track 0.00 -> 133.0 mm
- net /I/O19: track 0.00 -> 131.7 mm, vias 0 -> 1
- net /I/O20: track 0.00 -> 130.9 mm
- net /I/O12: track 0.00 -> 124.0 mm, vias 0 -> 1
- net /I/O6: track 0.00 -> 123.4 mm, vias 0 -> 1
- net /I/O7: track 0.00 -> 114.9 mm, vias 0 -> 1
- net /I/O8: track 0.00 -> 114.1 mm, vias 0 -> 1
- net /I/O14: track 0.00 -> 112.7 mm, vias 0 -> 1
- net /I/O13: track 0.00 -> 111.1 mm, vias 0 -> 1
- net /I/O10: track 0.00 -> 101.6 mm, vias 0 -> 1
- net /I/O11: track 0.00 -> 93.3 mm, vias 0 -> 1
- net /I/O3: track 0.00 -> 84.0 mm, vias 0 -> 1
- net /I/O2: track 0.00 -> 83.4 mm
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- added copper zone on B.Cu, net GND
- added copper zone on F.Cu, net GND
Other:
- board text added: "CPLD & STM32F030K Test Board made by GH Park @ 2026.01.27."

Commit message: 0215 artwork
Parts:
- removed the J2 at (119.5, 54.4)
- removed the R6 at (131.0, 53.0)
- added BT1: 3.7V, Connector_Molex:Molex_PicoBlade_53048-0210_1x02_P1.25mm_Horizontal, F.Cu at (123.0, 75.5)
- added C1: 47u, Capacitor_SMD:C_1206_3216Metric, F.Cu at (125.0, 60.0)
- added D1: Charge, LED_SMD:LED_0603_1608Metric, F.Cu at (119.5, 81.0)
- added D2: Standby, LED_SMD:LED_0603_1608Metric, F.Cu at (119.5, 82.5)
- added D3: RED, LED_SMD:LED_0603_1608Metric, F.Cu at (158.5, 93.5)
- added D4: RED, LED_SMD:LED_0603_1608Metric, F.Cu at (158.5, 96.1)
- added D5: RED, LED_SMD:LED_0603_1608Metric, F.Cu at (158.5, 98.5)
- added D6: RED, LED_SMD:LED_0603_1608Metric, F.Cu at (158.5, 101.0)
- added D7: RED, LED_SMD:LED_0603_1608Metric, F.Cu at (158.5, 103.5)
- added D8: RED, LED_SMD:LED_0603_1608Metric, F.Cu at (158.5, 106.0)
- added J1: USB_C_Receptacle_PowerOnly_6P, Connector_USB:USB_C_Receptacle_GCT_USB4125-xx-x-0190_6P_TopMnt_Horizontal, F.Cu at (119.5, 51.5)
- added J6: Microsemi_FlashPro-JTAG-10, Connector_IDC:IDC-Header_2x05_P2.54mm_Vertical, F.Cu at (122.7, 90.4)
- added R1: 1K5, Resistor_SMD:R_0603_1608Metric, F.Cu at (137.0, 54.0)
- added R10: 1K5, Resistor_SMD:R_0603_1608Metric, F.Cu at (165.5, 93.5)
- added R11: 1K5, Resistor_SMD:R_0603_1608Metric, F.Cu at (165.5, 96.0)
- added R12: 1K5, Resistor_SMD:R_0603_1608Metric, F.Cu at (165.5, 98.5)
- added R13: 1K5, Resistor_SMD:R_0603_1608Metric, F.Cu at (165.5, 101.0)
- added R14: 1K5, Resistor_SMD:R_0603_1608Metric, F.Cu at (165.5, 103.5)
- added R15: 1K5, Resistor_SMD:R_0603_1608Metric, F.Cu at (165.5, 106.0)
- added R16: 1K5, Resistor_SMD:R_0603_1608Metric, F.Cu at (162.0, 93.5)
- added R17: 1K5, Resistor_SMD:R_0603_1608Metric, F.Cu at (162.0, 96.0)
- added R18: 1K5, Resistor_SMD:R_0603_1608Metric, F.Cu at (162.0, 98.5)
- added R19: 1K5, Resistor_SMD:R_0603_1608Metric, F.Cu at (162.0, 101.0)
- added R2: 1K5, Resistor_SMD:R_0603_1608Metric, F.Cu at (137.0, 57.0)
- added R20: 1K5, Resistor_SMD:R_0603_1608Metric, F.Cu at (162.0, 103.5)
- added R21: 1K5, Resistor_SMD:R_0603_1608Metric, F.Cu at (162.0, 106.0)
- added R3: 5K1, Resistor_SMD:R_0603_1608Metric, F.Cu at (126.0, 52.5)
- added R4: 5K1, Resistor_SMD:R_0603_1608Metric, F.Cu at (126.0, 49.5)
- added SW1: SW_SPDT, fffff:SK12D07VG4NSPA_CNK, F.Cu at (119.0, 64.0)
- added U1: TP4056-42-ESOP8, Package_SO:SOIC-8-1EP_3.9x4.9mm_P1.27mm_EP2.41x3.3mm_ThermalVias, F.Cu at (131.5, 55.0)
- R5: value 5.1k -> 1K5; footprint Resistor_SMD:R_0603_1608Metric_Pad0.98x0.95mm_HandSolder -> Resistor_SMD:R_0603_1608Metric
- U4: value ATF1502ASV-xAx44 -> EPM3064ALC44-10N
- moved R5 5.01 mm to (126.0, 55.0), turned to -90 degrees
- moved R26 3.58 mm to (147.8, 62.5)
- moved R27 3.58 mm to (134.2, 63.2)
- moved R28 3.58 mm to (161.1, 62.5)
- moved SW3 3.58 mm to (141.5, 65.5)
- moved SW4 3.58 mm to (128.3, 65.5)
- moved SW5 3.58 mm to (155.0, 65.0)
- moved U4 3.26 mm to (145.3, 86.7)
- moved R8 2.54 mm to (164.0, 79.5)
- renumbered C1 to C2, C2 to C3, J1 to J2, J6 to J7, R10 to R22, R11 to R23, R12 to R24, R13 to R25, R7 to R26, R8 to R27, R9 to R28, R14 to R29, R15 to R30, R16 to R31, R17 to R32, R1 to R6, R2 to R7, R3 to R8, R4 to R9, SW1 to SW2, SW2 to SW3, SW3 to SW4, SW4 to SW5, U1 to U2, U2 to U3, U3 to U5
Connections:
- net /I/O1 renamed /I1
- net /I/O2 renamed /I2
- J5 pad 10: /I/O12 -> /IO14
- J5 pad 11: /I/O13 -> /IO16
- J5 pad 12: /I/O14 -> /IO18
- J5 pad 13: /I/O15 -> /IO19
- J5 pad 14: /I/O18 -> /IO20
- J5 pad 15: /I/O19 -> /IO21
- J5 pad 16: /I/O20 -> /IO24
- J5 pad 3: /I/O3 -> /IO4
- J5 pad 4: /I/O5 -> /IO5
- J5 pad 5: /I/O6 -> /IO6
- J5 pad 6: /I/O7 -> /IO8
- J5 pad 7: /I/O8 -> /IO9
- J5 pad 8: /I/O10 -> /IO11
- J5 pad 9: /I/O11 -> /IO12
- J7 pad 1: /I/O21 -> /IO25
- J7 pad 10: /I/O32 -> /IO39
- J7 pad 11: /I/O33 -> /IO40
- J7 pad 12: /I/O34 -> /I41
- J7 pad 13: /I/O35 -> /I43
- J7 pad 14: /I/O42 -> /I44
- J7 pad 15: /I/O43 -> unconnected-(J7-Pin_15-Pad15)
- J7 pad 16: /I/O44 -> unconnected-(J7-Pin_16-Pad16)
- J7 pad 2: /I/O22 -> /IO26
- J7 pad 3: /I/O23 -> /IO27
- J7 pad 4: /I/O25 -> /IO28
- J7 pad 5: /I/O26 -> /IO29
- J7 pad 6: /I/O27 -> /IO31
- J7 pad 7: /I/O28 -> /IO33
- J7 pad 8: /I/O30 -> /IO34
- J7 pad 9: /I/O31 -> /IO37
- R22 pad 1: /I/O6 -> /IO5
- R23 pad 1: /I/O7 -> /IO6
- R24 pad 1: /I/O8 -> /IO8
- R25 pad 1: /I/O10 -> /IO9
- R28 pad 2: /I/O3 -> /IO4
- R29 pad 1: /I/O11 -> /IO11
- R30 pad 1: /I/O12 -> /IO12
- R31 pad 1: /I/O13 -> /IO14
- R32 pad 1: /I/O14 -> /IO16
- SW5 pad 1: /I/O3 -> /IO4
- U4 pad 10: /I/O10 -> GND
- U4 pad 11: /I/O11 -> /IO11
- U4 pad 12: /I/O12 -> /IO12
- U4 pad 13: /I/O13 -> /TMS
- U4 pad 14: /I/O14 -> /IO14
- U4 pad 15: /I/O15 -> +3.3V
- U4 pad 16: GND -> /IO16
- U4 pad 17: +3.3V -> GND
- U4 pad 18: /I/O18 -> /IO18
- U4 pad 19: /I/O19 -> /IO19
- U4 pad 20: /I/O20 -> /IO20
- U4 pad 21: /I/O21 -> /IO21
- U4 pad 22: /I/O22 -> GND
- U4 pad 23: /I/O23 -> +3.3V
- U4 pad 24: GND -> /IO24
- U4 pad 25: /I/O25 -> /IO25
- U4 pad 26: /I/O26 -> /IO26
- U4 pad 27: /I/O27 -> /IO27
- U4 pad 28: /I/O28 -> /IO28
- U4 pad 29: +3.3V -> /IO29
- U4 pad 3: /I/O3 -> +3.3V
- U4 pad 30: /I/O30 -> GND
- U4 pad 31: /I/O31 -> /IO31
- U4 pad 32: /I/O32 -> /TCK
- U4 pad 33: /I/O33 -> /IO33
- U4 pad 34: /I/O34 -> /IO34
- U4 pad 35: /I/O35 -> +3.3V
- U4 pad 37: /I37 -> /IO37
- U4 pad 38: /I38 -> /TDO
- U4 pad 39: /I39 -> /IO39
- U4 pad 4: GND -> /IO4
- U4 pad 40: /I40 -> /IO40
- U4 pad 41: +3.3V -> /I41
- U4 pad 42: /I/O42 -> GND
- U4 pad 43: /I/O43 -> /I43
- U4 pad 44: /I/O44 -> /I44
- U4 pad 5: /I/O5 -> /IO5
- U4 pad 6: /I/O6 -> /IO6
- U4 pad 7: /I/O7 -> /TDI
- U4 pad 8: /I/O8 -> /IO8
- U4 pad 9: +3.3V -> /IO9
- U5 pad 12: /I/O15 -> /IO18
- U5 pad 6: /I/O20 -> /IO21
- U5 pad 8: /I/O19 -> /IO20
- U5 pad 9: /I/O18 -> /IO19
Routing:
- net /I/O18: track 140.0 -> 0.00 mm, vias 1 -> 0
- net /I/O15: track 133.0 -> 0.00 mm
- net /I/O19: track 131.7 -> 0.00 mm, vias 1 -> 0
- net /I/O20: track 130.9 -> 0.00 mm
- net /I/O12: track 124.0 -> 0.00 mm, vias 1 -> 0
- net /I/O6: track 123.4 -> 0.00 mm, vias 1 -> 0
- net /I/O7: track 114.9 -> 0.00 mm, vias 1 -> 0
- net /I/O8: track 114.1 -> 0.00 mm, vias 1 -> 0
- net /I/O14: track 112.7 -> 0.00 mm, vias 1 -> 0
- net /I/O13: track 111.1 -> 0.00 mm, vias 1 -> 0
- net /I/O10: track 101.6 -> 0.00 mm, vias 1 -> 0
- net /I/O11: track 93.3 -> 0.00 mm, vias 1 -> 0
- net /I/O3: track 84.0 -> 0.00 mm, vias 1 -> 0
- net /IO5: track 0.00 -> 73.5 mm
- net /IO8: track 0.00 -> 64.1 mm
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- removed copper zone on B.Cu, net GND
- removed copper zone on F.Cu, net GND

Commit message: 0218 artwork
Routing:
- net /IO20: track 57.8 -> 132.5 mm, vias 0 -> 1
- net /IO21: track 49.1 -> 120.0 mm, vias 0 -> 1
- net /I2: track 55.5 -> 121.3 mm, vias 0 -> 1
- net /IO18: track 47.2 -> 109.9 mm, vias 0 -> 1
- net /IO19: track 54.7 -> 112.8 mm, vias 1 -> 2
- net /IO16: track 49.1 -> 104.0 mm, vias 0 -> 1
- net /IO14: track 55.4 -> 108.1 mm, vias 0 -> 1
- net /IO12: track 54.5 -> 103.9 mm, vias 0 -> 1
- net +3.3V: track 391.0 -> 438.3 mm
- net /IO11: track 50.8 -> 96.7 mm, vias 0 -> 1
- net Net-(D1-K): track 0.00 -> 45.5 mm
- net /IO9: track 50.2 -> 93.3 mm, vias 0 -> 1
- net Vusb: track 17.7 -> 60.1 mm, vias 0 -> 2
- net Net-(D2-K): track 0.00 -> 39.9 mm
- net /IO4: track 48.7 -> 87.4 mm, vias 0 -> 1
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- added copper zone on B.Cu, net GND
- added copper zone on F.Cu, net GND
Other:
- board text added: "CPLD & STM32F030K Test Board made by GH Park @ 2026.02.15."
- board text removed: "CPLD & STM32F030K Test Board made by GH Park @ 2026.01.27."

Commit message: 0330 : SPLDTest save
Parts:
- removed D6: RED, LED_SMD:LED_0603_1608Metric
- removed J3, J5, J7: Conn_02x09_Top_Bottom, Connector_PinSocket_2.54mm:PinSocket_2x09_P2.54mm_Vertical
- removed R19: 1K5, Resistor_SMD:R_0603_1608Metric
- SW1: footprint fffff:SK12D07VG4NSPA_CNK -> Connector_Molex:Molex_Micro-Fit_3.0_43650-0315_1x03_P3.00mm_Vertical
- moved R13 4.03 mm to (169.5, 101.6)
- moved J4 2.45 mm to (211.0, 91.3)
- moved R6 2.45 mm to (199.8, 102.9)
- moved SW2 2.45 mm to (190.2, 94.6)
- moved D7 2.03 mm to (158.5, 101.5)
- moved D8 2.03 mm to (158.5, 104.0)
- moved R14 2.03 mm to (165.5, 101.5)
- moved R15 2.03 mm to (165.5, 104.0)
- moved R20 2.03 mm to (162.0, 101.5)
- moved R21 2.03 mm to (162.0, 104.0)
- moved SW1 0.58 mm to (119.0, 63.4)
Connections:
- U2 pad 14: Net-(J3-Pin_1) -> unconnected-(U2-PB0-Pad14)
- U2 pad 15: Net-(J3-Pin_2) -> unconnected-(U2-PB1-Pad15)
- U2 pad 26: Net-(J3-Pin_3) -> unconnected-(U2-PB3-Pad26)
- U2 pad 27: Net-(J3-Pin_4) -> unconnected-(U2-PB4-Pad27)
- U2 pad 28: Net-(J3-Pin_5) -> unconnected-(U2-PB5-Pad28)
- U2 pad 29: Net-(J3-Pin_6) -> unconnected-(U2-PB6-Pad29)
- U2 pad 30: Net-(J3-Pin_7) -> unconnected-(U2-PB7-Pad30)
- U2 pad 6: /PA0 -> unconnected-(U2-PA0-Pad6)
- U2 pad 7: /PA1 -> unconnected-(U2-PA1-Pad7)
- U4 pad 24: /IO24 -> unconnected-(U4-IO_C_33-Pad24)
- U4 pad 25: /IO25 -> unconnected-(U4-IO_C_35-Pad25)
- U4 pad 26: /IO26 -> unconnected-(U4-IO_C_36-Pad26)
- U4 pad 27: /IO27 -> unconnected-(U4-IO_C_37-Pad27)
- U4 pad 39: /IO39 -> unconnected-(U4-IO_D_57-Pad39)
- U4 pad 40: /IO40 -> unconnected-(U4-IO_D_62-Pad40)
- U4 pad 41: /I41 -> unconnected-(U4-IO_D_64-Pad41)
- U4 pad 43: /I43 -> unconnected-(U4-INPUT/GCLK1-Pad43)
- U4 pad 44: /I44 -> unconnected-(U4-INPUT/OE1-Pad44)
Routing:
- net +3.3V: track 438.3 -> 357.2 mm, vias 6 -> 3
- net /PA3: track 74.2 -> 13.0 mm
- net /PA2: track 69.1 -> 10.4 mm
- net /PA0: track 56.9 -> 0.00 mm
- net /PA1: track 56.2 -> 0.00 mm
- net /I44: track 49.5 -> 0.00 mm
- net /PA12: track 71.7 -> 22.3 mm, vias 3 -> 2
- net /PA11: track 67.2 -> 19.8 mm, vias 3 -> 0
- net /I2: track 121.3 -> 73.9 mm
- net /I43: track 46.3 -> 0.00 mm
- net /IO5: track 108.8 -> 63.1 mm
- net /I41: track 45.0 -> 0.00 mm
- net Net-(J3-Pin_6): track 41.1 -> 0.00 mm
- net Net-(J3-Pin_7): track 40.1 -> 0.00 mm
- net /IO4: track 87.4 -> 47.5 mm
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Other:
- board size 100 x 77 mm -> 100 x 70 mm
