File: SPLD_Test/SPLD_Test.kicad_sch (KiCad schematic)
At the start: 26 parts, among them J1 USB_C_Receptacle_PowerOnly_6P, J2 Conn_02x09_Top_Bottom, J3 Conn_02x09_Top_Bottom, J4 SPI OLED 1.3in, J5 SWD, J6 Conn_02x09_Top_Bottom, SW1 SW_MEC_5E, SW2 SW_MEC_5E, SW3 SW_MEC_5E, SW4 SW_MEC_5E, U1 ATF1502ASV-xAx44, U10 EA8105, U2 CA56-12CGKWA, U3 STM32F030K6Tx

Commit message: progress: CPLD Board complete
Parts:
- added R10, R11, R12, R13, R14, R15, R16, R17: 10k, Resistor_SMD:R_0402_1005Metric_Pad0.72x0.64mm_HandSolder, symbol Device:R
- C1: renamed from C9; now in the parts list
- C2: renamed from C1; now in the parts list
- J1: renamed from J4; footprint (none) -> Connector_PinSocket_2.54mm:PinSocket_1x07_P2.54mm_Vertical
- J3: renamed from J6; footprint (none) -> Connector_PinSocket_2.54mm:PinSocket_2x09_P2.54mm_Vertical
- J4: renamed from J5; footprint (none) -> Connector_PinSocket_2.54mm:PinSocket_1x06_P2.54mm_Vertical
- L1: renamed from L4; now in the parts list
- R1: renamed from R4; now in the parts list
- R2: renamed from R63; now in the parts list
- R3: renamed from R5; now in the parts list
- R4: renamed from R65; now in the parts list
- R5: renamed from R61; now in the parts list
- R6: renamed from R1; now in the parts list
- R7: renamed from R69; now in the parts list
- R8: renamed from R2; now in the parts list
- R9: renamed from R3; now in the parts list
- U2: renamed from U10; now in the parts list
- renumbered J1 to J2, J3 to J5, J2 to J6, SW4 to SW1, SW1 to SW3, SW3 to SW4, U3 to U1, U2 to U3, U1 to U4
Connections:
- net I/O10: now also R13.1; no longer U3.2 (d)
- net I/O11: now also R14.1; no longer U3.1 (e)
- net I/O12: now also R15.1; no longer U3.10 (f)
- net I/O13: now also R16.1; no longer U3.5 (g)
- net I/O14: now also R17.1; no longer U3.3 (DPX)
- net I/O6: now also R10.1; no longer U3.11 (a)
- net I/O7: now also R11.1; no longer U3.7 (b)
- net I/O8: now also R12.1; no longer U3.4 (c)
- new net: R11.2, U3.7 (b)
- new net: R10.2, U3.11 (a)
- new net: R16.2, U3.5 (g)
- new net: R14.2, U3.1 (e)
- new net: R12.2, U3.4 (c)
- new net: R15.2, U3.10 (f)
- new net: R13.2, U3.2 (d)
- new net: R17.2, U3.3 (DPX)
Other:
- moved on the sheet: U3

Commit message: progress: CPLD Big Change
Parts:
- removed U4: ATF1502ASV-xAx44, Package_LCC:PLCC-44_THT-Socket, symbol CPLD_Microchip:ATF1502ASV-xAx44
- added J7: Microsemi_FlashPro-JTAG-10, Connector_IDC:IDC-Header_2x05_P2.54mm_Vertical, symbol Connector:Microsemi_FlashPro-JTAG-10
- added U6: EPM3064ALC44-10N, Package_LCC:PLCC-44_THT-Socket, symbol GH_LIBRARIES:EPM3064ALC44-10N
Connections:
- net +3.3V: now also U6.15 (VCCIO(2.5VOR3.3V)), U6.23 (VCCINT(3.3VONLY)), U6.3 (VCCINT(3.3VONLY)), U6.35 (VCCIO(2.5VOR3.3V))
- net GND: now also U6.10 (GNDIO), U6.22 (GNDINT), U6.30 (GNDIO), U6.42 (GNDINT)
- net I37: now also U6.43 (INPUT/GCLK1)
- net I38: now also U6.44 (INPUT/OE1)
- net I39: now also U6.6 (IO_A_11)
- net I40: now also U6.5 (IO_A_14)
- net I/O1: now also U6.7 (TDI)
- net I/O10: now also U6.16 (IO_B_25)
- net I/O11: now also U6.17 (GNDIO)
- net I/O12: now also U6.18 (IO_B_21)
- net I/O13: now also U6.19 (IO_B_20)
- net I/O14: now also U6.20 (IO_B_19)
- net I/O15: now also U6.21 (IO_B_17)
- net I/O18: now also U6.24 (IO_C_33)
- net I/O19: now also U6.25 (IO_C_35)
- net I/O2: now also U6.8 (IO_A_5)
- net I/O20: now also U6.26 (IO_C_36)
- net I/O21: now also U6.27 (IO_C_37)
- net I/O22: now also U6.28 (IO_C_40)
- net I/O23: now also U6.29 (IO_C_41)
- net I/O25: now also U6.31 (IO_C_46)
- net I/O26: now also U6.32 (TCK)
- net I/O27: now also U6.33 (IO_D_49)
- net I/O28: now also U6.34 (IO_D_51)
- net I/O3: now also U6.9 (IO_A_4)
- net I/O30: now also U6.36 (GNDIO)
- net I/O31: now also U6.37 (IO_D_53)
- net I/O32: now also U6.38 (TDO)
- net I/O33: now also U6.39 (IO_D_57)
- net I/O34: now also U6.40 (IO_D_62)
- net I/O35: now also U6.41 (IO_D_64)
- net I/O42: now also U6.4 (IO_A_16)
- net I/O43: now also U6.2 (INPUT/OE2/GCLK2)
- net I/O44: now also U6.1 (INPUT/GCLRN)
- net I/O5: now also U6.11 (IO_A_3)
- net I/O6: now also U6.12 (IO_A_1)
- net I/O7: now also U6.13 (TMS)
- net I/O8: now also U6.14 (IO_B_30)
- new net: J7.10 (GND), J7.2 (GND)
Other:
- note added: "여기다가 그거 충전회로와 5V 승압회로 만들어서 적용하기 JTAG 만들어서 적용하기 here we should make charging circuit and JTAG circuit"

Commit message: 0215 artwork
Parts:
- removed J2: USB_C_Receptacle_PowerOnly_6P, Connector_USB:USB_C_Receptacle_HRO_TYPE-C-31-M-17, symbol Connector:USB_C_Receptacle_PowerOnly_6P
- removed J7: Microsemi_FlashPro-JTAG-10, Connector_IDC:IDC-Header_2x05_P2.54mm_Vertical, symbol Connector:Microsemi_FlashPro-JTAG-10
- removed R6: 5.1k, Resistor_SMD:R_0603_1608Metric_Pad0.98x0.95mm_HandSolder, symbol Device:R
- added BT1: 3.7V, Connector_Molex:Molex_PicoBlade_53048-0210_1x02_P1.25mm_Horizontal, symbol Device:Battery_Cell
- added C1: 47u, Capacitor_SMD:C_1206_3216Metric, symbol Device:C
- added D1: Charge, LED_SMD:LED_0603_1608Metric, symbol Device:LED_Small
- added D2: Standby, LED_SMD:LED_0603_1608Metric, symbol Device:LED_Small
- added D3, D4, D5, D6, D7, D8: RED, LED_SMD:LED_0603_1608Metric, symbol Device:LED_Small
- added J1: USB_C_Receptacle_PowerOnly_6P, Connector_USB:USB_C_Receptacle_GCT_USB4125-xx-x-0190_6P_TopMnt_Horizontal, symbol Connector:USB_C_Receptacle_PowerOnly_6P
- added J6: Microsemi_FlashPro-JTAG-10, Connector_IDC:IDC-Header_2x05_P2.54mm_Vertical, symbol Connector:Microsemi_FlashPro-JTAG-10
- added R1, R10, R11, R12, R13, R14, R15, R16, R17, R18, R19, R2, R20, R21: 1K5, Resistor_SMD:R_0603_1608Metric, symbol Device:R
- added R3, R4: 5K1, Resistor_SMD:R_0603_1608Metric, symbol Device:R
- added SW1: SW_SPDT, SK12D07VG4NSPA_CNK, symbol Switch:SW_SPDT
- added U1: TP4056-42-ESOP8, Package_SO:SOIC-8-1EP_3.9x4.9mm_P1.27mm_EP2.41x3.3mm_ThermalVias, symbol Battery_Management:TP4056-42-ESOP8
- R5: value 5.1k -> 1K5; footprint Resistor_SMD:R_0603_1608Metric_Pad0.98x0.95mm_HandSolder -> Resistor_SMD:R_0603_1608Metric; LCSC (none) -> C22843
- renumbered C1 to C2, C2 to C3, J1 to J2, J6 to J7, R10 to R22, R11 to R23, R12 to R24, R13 to R25, R7 to R26, R8 to R27, R9 to R28, R14 to R29, R15 to R30, R16 to R31, R17 to R32, R1 to R6, R2 to R7, R3 to R8, R4 to R9, SW1 to SW2, SW2 to SW3, SW3 to SW4, SW4 to SW5, U1 to U2, U2 to U3, U6 to U4, U3 to U5
Connections:
- net +3.3V: now also J6.4 (VccTRGT)
- net +5V: now also SW1.1 (A)
- net GND: now also U4.17 (GNDIO), U4.36 (GNDIO), BT1.2 (-), C1.1, J1.A12 (GND), J1.B12 (GND), J1.S1 (SHIELD), J6.10 (GND), J6.2 (GND), R16.1, R17.1, R18.1, R19.1, R20.1, R21.1, R3.2, R4.2, U1.1 (TEMP), U1.3 (GND), U1.9 (EPAD)
- net PA10: now also R12.1
- net PA11: now also R13.1
- net PA12: now also R14.1
- net PA15: now also R15.1
- net PA2: now also R10.1
- net PA3: now also R11.1
- net at R5.1: now also U1.2 (PROG)
- net I37 renamed I43
- net I43: now also J7.13 (Pin_13)
- net I38 renamed I44
- net I44: now also J7.14 (Pin_14)
- net I39 renamed IO6
- net IO6: now also J5.5 (Pin_5), R23.1
- net I40 renamed IO5
- net IO5: now also J5.4 (Pin_4), R22.1
- net I/O1 renamed I1
- net I1: now also U4.1 (INPUT/GCLRN); no longer U4.7 (TDI)
- removed net I/O10: J5.8 (Pin_8), R25.1, U4.16 (IO_B_25)
- removed net I/O11: J5.9 (Pin_9), R29.1, U4.17 (GNDIO)
- removed net I/O12: J5.10 (Pin_10), R30.1, U4.18 (IO_B_21)
- removed net I/O13: J5.11 (Pin_11), R31.1, U4.19 (IO_B_20)
- removed net I/O14: J5.12 (Pin_12), R32.1, U4.20 (IO_B_19)
- removed net I/O15: J5.13 (Pin_13), U4.21 (IO_B_17), U5.12 (CA1)
- removed net I/O18: J5.14 (Pin_14), U4.24 (IO_C_33), U5.9 (CA2)
- removed net I/O19: J5.15 (Pin_15), U4.25 (IO_C_35), U5.8 (CA3)
- net I/O2 renamed I2
- net I2: now also U4.2 (INPUT/OE2/GCLK2); no longer U4.8 (IO_A_5)
- removed net I/O20: J5.16 (Pin_16), U4.26 (IO_C_36), U5.6 (CA4)
- net I/O21 renamed IO25
- net IO25: now also U4.25 (IO_C_35); no longer U4.27 (IO_C_37)
- net I/O22 renamed IO26
- net IO26: now also U4.26 (IO_C_36); no longer U4.28 (IO_C_40)
- net I/O23 renamed IO27
- net IO27: now also U4.27 (IO_C_37); no longer U4.29 (IO_C_41)
- net I/O25 renamed IO28
- net IO28: now also U4.28 (IO_C_40), D3.2 (A), R10.2; no longer U4.31 (IO_C_46)
- net I/O26 renamed IO29
- net IO29: now also U4.29 (IO_C_41), D4.2 (A), R11.2; no longer U4.32 (TCK)
- net I/O27 renamed IO31
- net IO31: now also U4.31 (IO_C_46), D5.2 (A), R12.2; no longer U4.33 (IO_D_49)
- net I/O28 renamed IO33
- net IO33: now also U4.33 (IO_D_49), D6.2 (A), R13.2; no longer U4.34 (IO_D_51)
- net I/O3 renamed IO4
- net IO4: now also U4.4 (IO_A_16); no longer U4.9 (IO_A_4)
- net I/O30 renamed IO34
- net IO34: now also U4.34 (IO_D_51), D7.2 (A), R14.2; no longer U4.36 (GNDIO)
- net I/O31 renamed IO37
- net IO37: now also D8.2 (A), R15.2
- net I/O32 renamed IO39
- net IO39: now also U4.39 (IO_D_57); no longer U4.38 (TDO)
- net I/O33 renamed IO40
- net IO40: now also U4.40 (IO_D_62); no longer U4.39 (IO_D_57)
- net I/O34 renamed I41
- net I41: now also U4.41 (IO_D_64); no longer U4.40 (IO_D_62)
- removed net I/O35: J7.13 (Pin_13), U4.41 (IO_D_64)
- removed net I/O42: J7.14 (Pin_14), U4.4 (IO_A_16)
- net I/O43: no longer names the net of J7.15 (Pin_15)
- net I/O43: no longer U4.2 (INPUT/OE2/GCLK2)
- net I/O44: no longer names the net of J7.16 (Pin_16)
- net I/O44: no longer U4.1 (INPUT/GCLRN)
- net I/O5 renamed IO11
- net IO11: now also J5.8 (Pin_8), R29.1; no longer J5.4 (Pin_4)
- removed net I/O6: J5.5 (Pin_5), R22.1, U4.12 (IO_A_1)
- removed net I/O7: J5.6 (Pin_6), R23.1, U4.13 (TMS)
- removed net I/O8: J5.7 (Pin_7), R24.1, U4.14 (IO_B_30)
- new net: D2.1 (K), R2.2
- new net: J1.B5 (CC2), R3.1
- new net: D3.1 (K), R16.2
- new net: J1.A5 (CC1), R4.1
- new net: D5.1 (K), R18.2
- new net: R2.1, U1.6 (~{STDBY})
- new net: R1.1, U1.7 (~{CHRG})
- new net: D6.1 (K), R19.2
- new net: D4.1 (K), R17.2
- new net: D1.1 (K), R1.2
- new net: D7.1 (K), R20.2
- new net: D8.1 (K), R21.2
- new net IO12: J5.9 (Pin_9), R30.1, U4.12 (IO_A_1)
- new net IO14: J5.10 (Pin_10), R31.1, U4.14 (IO_B_30)
- new net IO16: J5.11 (Pin_11), R32.1, U4.16 (IO_B_25)
- new net IO18: J5.12 (Pin_12), U4.18 (IO_B_21), U5.12 (CA1)
- new net IO19: J5.13 (Pin_13), U4.19 (IO_B_20), U5.9 (CA2)
- new net IO20: J5.14 (Pin_14), U4.20 (IO_B_19), U5.8 (CA3)
- new net IO21: J5.15 (Pin_15), U4.21 (IO_B_17), U5.6 (CA4)
- new net IO24: J5.16 (Pin_16), U4.24 (IO_C_33)
- new net IO8: J5.6 (Pin_6), R24.1, U4.8 (IO_A_5)
- new net IO9: J5.7 (Pin_7), R25.1, U4.9 (IO_A_4)
- new net TCK: J6.1 (TCK), U4.32 (TCK)
- new net TDI: J6.3 (TDO), U4.7 (TDI)
- new net TDO: J6.9 (TDI), U4.38 (TDO)
- new net TMS: J6.5 (TMS), U4.13 (TMS)
- new net Vbat: BT1.1 (+), C1.2, SW1.2 (B), U1.5 (BAT)
- new net Vusb: D1.2 (A), D2.2 (A), J1.A9 (VBUS), J1.B9 (VBUS), U1.4 (V_{CC}), U1.8 (CE)
- no-connect marks 0 -> 3
Other:
- note added: "1K5 = 0.8A"
- moved on the sheet: C2, C3, L1, R7, R9, U3

Commit message: 0330 : SPLDTest save
Parts:
- removed C1: 47u, Capacitor_SMD:C_1206_3216Metric, symbol Device:C
- removed D6: RED, LED_SMD:LED_0603_1608Metric, symbol Device:LED_Small
- removed J2: SPI OLED 1.3in, Connector_PinSocket_2.54mm:PinSocket_1x07_P2.54mm_Vertical, symbol Connector:Conn_01x07_Socket
- removed J3, J5, J7: Conn_02x09_Top_Bottom, Connector_PinSocket_2.54mm:PinSocket_2x09_P2.54mm_Vertical, symbol Connector_Generic:Conn_02x09_Top_Bottom
- removed R19: 1K5, Resistor_SMD:R_0603_1608Metric, symbol Device:R
- removed U4: EPM3064ALC44-10N, Package_LCC:PLCC-44_THT-Socket, symbol GH_LIBRARIES:EPM3064ALC44-10N
- added C3: 47u, Capacitor_SMD:CP_Elec_6.3x5.7, symbol Device:C_Polarized
- added J5: 0.96inch OLED, Connector_PinSocket_2.54mm:PinSocket_1x04_P2.54mm_Vertical, symbol Connector:Conn_01x04_Socket
- added U3: EPM3064ALC44-10N, Package_LCC:PLCC-44_THT-Socket, symbol ul_EPM3064ALC44-10N:EPM3064ALC44-10N
- BT1: Component Name (none) -> Battery_Cell
- C1: renamed from C3; Component Name (none) -> CAP POL
- C2: Component Name (none) -> CAP POL
- D1, D2, D3, D4, D5: Component Name (none) -> LED
- D6: renamed from D7; Component Name (none) -> LED
- D7: renamed from D8; Component Name (none) -> LED
- J1: Component Name (none) -> USB_C_Receptacle_PowerOnly_6P
- J2: renamed from J6; Component Name (none) -> Microsemi_FlashPro-JTAG-10
- J4: Component Name (none) -> CONN_01x06_Socket
- L1: Component Name (none) -> L
- R1: renamed from R3; Component Name (none) -> R
- R10: renamed from R12; Component Name (none) -> R
- R11: renamed from R13; Component Name (none) -> R
- R12: renamed from R14; Component Name (none) -> R
- R13: renamed from R15; Component Name (none) -> R
- R14: renamed from R6; Component Name (none) -> R
- R15: renamed from R16; Component Name (none) -> R
- R16: renamed from R17; Component Name (none) -> R
- R17: renamed from R18; Component Name (none) -> R
- R18: renamed from R20; Component Name (none) -> R
- R19: renamed from R21; Component Name (none) -> R
- R2: renamed from R4; Component Name (none) -> R
- R20: renamed from R8; Component Name (none) -> R
- R21: renamed from R26; Component Name (none) -> R
- R22, R23, R24, R25, R5: Component Name (none) -> R
- R26: renamed from R29; Component Name (none) -> R
- R27: renamed from R30; Component Name (none) -> R
- R28: renamed from R31; Component Name (none) -> R
- R29: renamed from R32; Component Name (none) -> R
- R3: renamed from R1; Component Name (none) -> R
- R30: renamed from R27; Component Name (none) -> R
- R31: renamed from R28; Component Name (none) -> R
- R4: renamed from R2; Component Name (none) -> R
- R6: renamed from R7; value 2.35k -> 22k; footprint Resistor_SMD:R_0402_1005Metric_Pad0.72x0.64mm_HandSolder -> Resistor_SMD:R_0603_1608Metric; Component Name (none) -> R
- R7: renamed from R9; value 76.9R -> 750R; Component Name (none) -> R
- R8: renamed from R10; Component Name (none) -> R
- R9: renamed from R11; Component Name (none) -> R
- SW1: footprint SK12D07VG4NSPA_CNK -> Connector_Molex:Molex_Micro-Fit_3.0_43650-0315_1x03_P3.00mm_Vertical; Component Name (none) -> SW_SPDT
- SW2: value SW_MEC_5E -> SW_SPST; Component Name (none) -> SW_PUSH
- SW3, SW4, SW5: Component Name (none) -> SW_PUSH
- U1: renamed from U3; Component Name (none) -> TPS62A01APDDC
- U2: renamed from U1; Component Name (none) -> TP4056-42-ESOP8
- U4: renamed from U2; Component Name (none) -> STM32F030K6Tx
- U5: Component Name (none) -> CA56-12CGKWA
Connections:
- net +3.3V: now also J5.2 (Pin_2), U3.15 (VCCIO(2.5VOR3.3V)), U3.23 (VCCINT(3.3VONLY)), U3.3 (VCCINT(3.3VONLY)), U3.35 (VCCIO(2.5VOR3.3V))
- net GND: now also C3.2, J5.1 (Pin_1), U3.10 (GNDIO), U3.17 (GNDIO), U3.22 (GNDINT), U3.30 (GNDIO), U3.36 (GNDIO), U3.42 (GNDINT)
- net I1: now also U3.1 (INPUT/GCLRN)
- net I2: now also U3.2 (INPUT/OE2/GCLK2)
- net IO11: now also U3.11 (IO_A_3)
- net IO12: now also U3.12 (IO_A_1)
- net IO14: now also U3.14 (IO_B_30)
- net IO16: now also U3.16 (IO_B_25)
- net IO18: now also U3.18 (IO_B_21)
- net IO19: now also U3.19 (IO_B_20)
- net IO20: now also U3.20 (IO_B_19)
- net IO21: now also U3.21 (IO_B_17)
- net IO28: now also U3.28 (IO_C_40)
- net IO29: now also U3.29 (IO_C_41)
- net IO31: now also U3.31 (IO_C_46)
- net IO33: now also U3.33 (IO_D_49)
- net IO34: now also U3.34 (IO_D_51)
- net IO37: now also U3.37 (IO_D_53)
- net IO4: now also U3.4 (IO_A_16)
- net IO5: now also U3.5 (IO_A_14)
- net IO6: now also U3.6 (IO_A_11)
- net IO8: now also U3.8 (IO_A_5)
- net IO9: now also U3.9 (IO_A_4)
- net TCK: now also U3.32 (TCK)
- net TDI: now also J2.9 (TDI), U3.7 (TDI); no longer J2.3 (TDO)
- net TDO: now also J2.3 (TDO), U3.38 (TDO); no longer J2.9 (TDI)
- net TMS: now also U3.13 (TMS)
- net Vbat: now also C3.1
- net SCL: now reaches U4.29 (PB6)
- net SCL: now also J5.3 (Pin_3)
- net SDA: now reaches U4.30 (PB7)
- net SDA: now also J5.4 (Pin_4)
- net CLK: no longer names the net of U4.11 (PA5)
- net DC: no longer names the net of U4.19 (PA9)
- net MOSI: no longer names the net of U4.13 (PA7)
- net NSS: no longer names the net of U4.10 (PA4)
- net OLEDRST: no longer names the net of U4.18 (PA8)
- net PA0: no longer names the net of U4.6 (PA0)
- net PA1: no longer names the net of U4.7 (PA1)
- no-connect marks 3 -> 29
Other:
- note added: "3.7V to 3.3V Buck Convertor"
- note added: "7-segment 4digits"
- note added: "CPLD - STM32 Connections"
- note added: "CPLD - STM32 Connections Status Check LED"
- note added: "CPLD Chip"
- note added: "JTAG Programmer Socket"
- note added: "LiPo Battery Charger"
- note added: "STM32 Circuits"
- note removed: "여기다가 그거 충전회로와 5V 승압회로 만들어서 적용하기 JTAG 만들어서 적용하기 here we should make charging circuit and JTAG circuit"
- moved on the sheet: BT1, C1, C2, D1, D2, D3, D4, D5, D6, D7, J1, J2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
