File: kalimba_V2/kalimba.kicad_sch (KiCad schematic)
At the start: 25 parts, among them J2 Conn_01x08, J3 Conn_01x08, SW1 SW_SPDT, U1 WS2812B-2020, U10 WS2812B-2020, U11 WS2812B-2020, U12 WS2812B-2020, U13 WS2812B-2020, U14 WS2812B-2020, U15 WS2812B-2020, U16 WS2812B-2020, U17 WS2812B-2020, U18 WS2812B-2020, U19 WS2812B-2020, U2 WS2812B-2020, U20 WS2812B-2020, U21 WS2812B-2020, U3 WS2812B-2020, U4 WS2812B-2020, U5 WS2812B-2020, U6 WS2812B-2020, U7 WS2812B-2020, U8 WS2812B-2020, U9 WS2812B-2020

Commit message: hey
Parts:
- removed J2, J3: Conn_01x08, Connector_PinSocket_2.54mm:PinSocket_1x08_P2.54mm_Vertical, symbol Connector_Generic:Conn_01x08
- added C1: 100nF, Capacitor_SMD:C_0402_1005Metric, symbol Device:C
- added R1: 330R, Resistor_SMD:R_0402_1005Metric, symbol Device:R
- added U1: AMS1117-3.3, Package_TO_SOT_SMD:SOT-223-3_TabPin2, symbol Regulator_Linear:AMS1117-3.3
- added U2: ESP32-WROOM-32E, RF_Module:ESP32-WROOM-32D, symbol RF_Module:ESP32-WROOM-32E
- renumbered U8 to U10, U9 to U11, U10 to U12, U11 to U13, U12 to U14, U13 to U15, U14 to U16, U15 to U17, U16 to U18, U17 to U19, U18 to U20, U19 to U21, U20 to U22, U21 to U23, U1 to U3, U2 to U4, U3 to U5, U4 to U6, U5 to U7, U6 to U8, U7 to U9
Connections:
- net +5V: now also U1.3 (VI)
- net GND: now also C1.2, U1.1 (GND), U2.1 (GND), U2.15 (GND), U2.38 (GND), U2.39 (GND)
- net usb Serial/Vusb: now reaches BT1.1 (+), SW1.2 (B)
- net at U23.3 (DI): now also R1.2
- new net: R1.1, U2.27 (IO16)
- new net IO0: U2.25 (IO0)
- new net RXD: U2.34 (RXD0/IO3)
- new net TXD: U2.35 (TXD0/IO1)
- new net usb Serial/3V3: C1.1, U1.2 (VO), U2.2 (VDD)
- new net usb Serial/EN: U2.3 (EN)
Other:
- added sheet usb Serial (untitled.kicad_sch)
- moved on the sheet: BT1, SW1
